File: kicad/LotusCharger.kicad_pcb (KiCad board)
At the start: 2 copper layers, 53.3 x 24.1 mm, 10 parts, among them P1 Solar Panel, P2 Battery

Commit message: Layout finished and sending to Fab.
Parts:
- added G***: LOGO, tl2c-footprint:MyBasic_rounded_50_1, F.Cu at (141.6, 116.8)
- added LGO***: LOGO, tl2c-footprint:KiCad-Logo, F.Cu at (167.6, 118.1)
- added P3: Load Power, tl2c-footprint:PCB_Screw_Terminal_Block_5.08mm_x_2, F.Cu at (153.7, 101.0)
- added P4: Load, tl2c-footprint:PCB_Screw_Terminal_Block_5.08mm_x_2, F.Cu at (163.8, 101.0)
- added P5: Battery Monitor, Terminal_Blocks:TerminalBlock_Pheonix_MPT-2.54mm_2pol, F.Cu at (169.5, 99.1)
- added P6: Cell Monitor, Terminal_Blocks:TerminalBlock_Pheonix_MPT-2.54mm_2pol, F.Cu at (142.9, 99.1)
- D2: moved to B.Cu
- P1, P2: footprint Terminal_Blocks:TerminalBlock_4UCON_19963_02x3.5mm_Straight -> tl2c-footprint:PCB_Screw_Terminal_Block_5.08mm_x_2
- moved D1 7.75 mm to (149.2, 108.0)
- moved D2 7.10 mm to (166.4, 112.4)
- moved D3 7.10 mm to (154.3, 118.1)
- moved D4 6.63 mm to (159.4, 108.0)
- moved P2 1.80 mm to (175.3, 110.5)
- moved REF** 1.27 mm to (179.1, 116.8)
- moved REF** 1.27 mm to (133.3, 116.8)
- moved REF** 1.27 mm to (179.1, 97.8)
- moved REF** 1.27 mm to (133.3, 97.8)
- moved P1 0.64 mm to (136.5, 105.4)
Connections:
- net Net-(D1-Pad2) renamed /VIn
- net Net-(D2-Pad1) renamed /VOut
Routing:
- net /VOut: track 20.8 -> 42.0 mm
- net /VIn: track 33.4 -> 47.0 mm
- net Net-(P3-Pad1): track 0.00 -> 5.08 mm
- net Net-(D3-Pad1): track 6.35 -> 5.08 mm
- net Net-(D1-Pad1): track 6.35 -> 5.08 mm
Other:
- board size 53.3 x 24.1 mm -> 53.3 x 26.7 mm
- rule pad_to_mask_clearance: 0.2 -> 0
- board text added: "+ -"
- board text added: "Batt Mon"
- board text added: "Battery"
- board text added: "Charging"
- board text added: "Load + -"
- board text added: "Load Power + -"
- board text added: "Lotus Charger 2L_1 Input: 9V 109mA Solar Output: 6V 1.2Ah Sealed Lead Acid"
- board text added: "Solar Mon"
- board text added: "Solar Panel"
