File: kicad/LotusCharger.sch (KiCad schematic (older format))
At the start: 6 parts, among them P1 Solar Panel, P2 Battery

Commit message: Layout finished and sending to Fab.
Parts:
- added P3: Load Power, tl2c-footprint:PCB_Screw_Terminal_Block_5.08mm_x_2, symbol CONN_01X02
- added P4: Load, tl2c-footprint:PCB_Screw_Terminal_Block_5.08mm_x_2, symbol CONN_01X02
- added P5: Battery Monitor, Terminal_Blocks:TerminalBlock_Pheonix_MPT-2.54mm_2pol, symbol CONN_01X02
- added P6: Cell Monitor, Terminal_Blocks:TerminalBlock_Pheonix_MPT-2.54mm_2pol, symbol CONN_01X02
- P1, P2: footprint Terminal_Blocks:TerminalBlock_4UCON_19963_02x3.5mm_Straight -> tl2c-footprint:PCB_Screw_Terminal_Block_5.08mm_x_2
Connections:
- net GND: now also P4.1 (P1), P5.1 (P1), P6.1 (P1)
- net VIn: now reaches D1.2 (A), D2.2 (A), P1.1 (P1)
- net VIn: now also P6.2 (P2)
- net VOut: now reaches D2.1 (K), D4.1 (K), P2.2 (P2)
- net VOut: now also P3.2 (P2), P5.2 (P2)
- new net: P3.1 (P1), P4.2 (P2)
Other:
- moved on the sheet: D1, D2, D3, D4, P1, P2
Changed lines of the file:
@@
 LIBS:contrib
 LIBS:valves
+LIBS:tl2c-symbols
+LIBS:LotusCharger-cache
 EELAYER 25 0
 EELAYER END
@@
 L D D1
 U 1 1 59BD4547
-P 3700 2150
-F 0 "D1" H 3700 2250 50  0000 C CNN
-F 1 "IN4004" H 3700 2050 50  0000 C CNN
-F 2 "Diodes_ThroughHole:D_DO-41_SOD81_P10.16mm_Horizontal" H 3700 2150 60  0001 C CNN
-F 3 "" H 3700 2150 60  0000 C CNN
-F 4 "Value" H 3700 2150 60  0001 C CNN "Link"
-	1    3700 2150
+P 5100 2000
+F 0 "D1" H 5100 2100 50  0000 C CNN
+F 1 "IN4004" H 5100 1900 50  0000 C CNN
+F 2 "Diodes_ThroughHole:D_DO-41_SOD81_P10.16mm_Horizontal" H 5100 2000 60  0001 C CNN
+F 3 "" H 5100 2000 60  0000 C CNN
+F 4 "Value" H 5100 2000 60  0001 C CNN "Link"
+	1    5100 2000
 	-1   0    0    1
 $EndComp
@@
 L D D3
 U 1 1 59BD45D9
-P 4250 2150
-F 0 "D3" H 4250 2250 50  0000 C CNN
-F 1 "IN4004" H 4250 2050 50  0000 C CNN
-F 2 "Diodes_ThroughHole:D_DO-41_SOD81_P10.16mm_Horizontal" H 4250 2150 60  0001 C CNN
-F 3 "" H 4250 2150 60  0000 C CNN
-F 4 "Value" H 4250 2150 60  0001 C CNN "Link"
-	1    4250 2150
+P 5650 2000
+F 0 "D3" H 5650 2100 50  0000 C CNN
+F 1 "IN4004" H 5650 1900 50  0000 C CNN
+F 2 "Diodes_ThroughHole:D_DO-41_SOD81_P10.16mm_Horizontal" H 5650 2000 60  0001 C CNN
+F 3 "" H 5650 2000 60  0000 C CNN
+F 4 "Value" H 5650 2000 60  0001 C CNN "Link"
+	1    5650 2000
 	-1   0    0    1
 $EndComp
@@
 L D D4
 U 1 1 59BD4623
-P 4750 2150
-F 0 "D4" H 4750 2250 50  0000 C CNN
-F 1 "IN4004" H 4750 2050 50  0000 C CNN
-F 2 "Diodes_ThroughHole:D_DO-41_SOD81_P10.16mm_Horizontal" H 4750 2150 60  0001 C CNN
-F 3 "" H 4750 2150 60  0000 C CNN
-F 4 "Value" H 4750 2150 60  0001 C CNN "Link"
-	1    4750 2150
+P 6150 2000
+F 0 "D4" H 6150 2100 50  0000 C CNN
+F 1 "IN4004" H 6150 1900 50  0000 C CNN
+F 2 "Diodes_ThroughHole:D_DO-41_SOD81_P10.16mm_Horizontal" H 6150 2000 60  0001 C CNN
+F 3 "" H 6150 2000 60  0000 C CNN
+F 4 "Value" H 6150 2000 60  0001 C CNN "Link"
+	1    6150 2000
 	-1   0    0    1
 $EndComp
@@
 L LED D2
 U 1 1 59BD4664
-P 4250 1700
-F 0 "D2" H 4250 1800 50  0000 C CNN
-F 1 "LED" H 4250 1600 50  0000 C CNN
-F 2 "LEDs:LED_D5.0mm" H 4250 1700 60  0001 C CNN
-F 3 "" H 4250 1700 60  0000 C CNN
-	1    4250 1700
+P 5650 1550
+F 0 "D2" H 5650 1650 50  0000 C CNN
+F 1 "LED" H 5650 1450 50  0000 C CNN
+F 2 "LEDs:LED_D5.0mm" H 5650 1550 60  0001 C CNN
+F 3 "" H 5650 1550 60  0000 C CNN
+	1    5650 1550
 	-1   0    0    1
 $EndComp
@@
 L CONN_01X02 P1
 U 1 1 59BD46AD
-P 2550 2200
-F 0 "P1" H 2550 2350 50  0000 C CNN
-F 1 "Solar Panel" V 2650 2200 50  0000 C CNN
-F 2 "Terminal_Blocks:TerminalBlock_4UCON_19963_02x3.5mm_Straight" H 2550 2200 60  0001 C CNN
-F 3 "" H 2550 2200 60  0000 C CNN
-	1    2550 2200
+P 3950 2050
+F 0 "P1" H 3950 2200 50  0000 C CNN
+F 1 "Solar Panel" V 4050 2050 50  0000 C CNN
+F 2 "tl2c-footprint:PCB_Screw_Terminal_Block_5.08mm_x_2" H 3950 2050 60  0001 C CNN
+F 3 "" H 3950 2050 60  0000 C CNN
+	1    3950 2050
 	-1   0    0    -1
 $EndComp
@@
 L GND #PWR01
 U 1 1 59BD4734
-P 2900 2700
-F 0 "#PWR01" H 2900 2450 50  0001 C CNN
-F 1 "GND" H 2900 2550 50  0000 C CNN
-F 2 "" H 2900 2700 60  0000 C CNN
-F 3 "" H 2900 2700 60  0000 C CNN
-	1    2900 2700
-	1    0    0    -1
-$EndComp
-Wire Wire Line
-	2750 2250 2900 2250
-Wire Wire Line
-	2900 2250 2900 2700
-Wire Wire Line
-	2750 2150 3550 2150
-Wire Wire Line
-	3850 2150 4100 2150
-Wire Wire Line
-	4400 2150 4600 2150
-Wire Wire Line
-	4900 2150 5800 2150
+P 4300 2550
+F 0 "#PWR01" H 4300 2300 50  0001 C CNN
+F 1 "GND" H 4300 2400 50  0000 C CNN
+F 2 "" H 4300 2550 60  0000 C CNN
+F 3 "" H 4300 2550 60  0000 C CNN
+	1    4300 2550
+	1    0    0    -1
+$EndComp
 $Comp
 L GND #PWR02
 U 1 1 59BD4787
-P 5650 2700
-F 0 "#PWR02" H 5650 2450 50  0001 C CNN
-F 1 "GND" H 5650 2550 50  0000 C CNN
-F 2 "" H 5650 2700 60  0000 C CNN
-F 3 "" H 5650 2700 60  0000 C CNN
-	1    5650 2700
-	1    0    0    -1
-$EndComp
-Wire Wire Line
-	4450 1700 5050 1700
-Wire Wire Line
-	5050 1700 5050 2150
-Connection ~ 5050 2150
-Wire Wire Line
-	4050 1700 3400 1700
-Wire Wire Line
-	3400 1700 3400 2150
-Connection ~ 3400 2150
+P 7050 2550
+F 0 "#PWR02" H 7050 2300 50  0001 C CNN
+F 1 "GND" H 7050 2400 50  0000 C CNN
+F 2 "" H 7050 2550 60  0000 C CNN
+F 3 "" H 7050 2550 60  0000 C CNN
+	1    7050 2550
+	1    0    0    -1
+$EndComp
 $Comp
 L CONN_01X02 P2
 U 1 1 59BD47DC
-P 6000 2200
-F 0 "P2" H 6000 2350 50  0000 C CNN
-F 1 "Battery" V 6100 2200 50  0000 C CNN
-F 2 "Terminal_Blocks:TerminalBlock_4UCON_19963_02x3.5mm_Straight" H 6000 2200 60  0001 C CNN
-F 3 "" H 6000 2200 60  0000 C CNN
-	1    6000 2200
-	1    0    0    1
-$EndComp
-Wire Wire Line
-	5800 2250 5650 2250
-Wire Wire Line
-	5650 2250 5650 2700
+P 7400 2050
+F 0 "P2" H 7400 2200 50  0000 C CNN
+F 1 "Battery" V 7500 2050 50  0000 C CNN
+F 2 "tl2c-footprint:PCB_Screw_Terminal_Block_5.08mm_x_2" H 7400 2050 60  0001 C CNN
+F 3 "" H 7400 2050 60  0000 C CNN
+	1    7400 2050
+	1    0    0    1
+$EndComp
+Text Label 6850 2000 0    60   ~ 0
+VOut
+Text Label 4350 2000 0    60   ~ 0
+VIn
+$Comp
+L CONN_01X02 P5
+U 1 1 59BE39F3
+P 4500 3150
+F 0 "P5" H 4500 3300 50  0000 C CNN
+F 1 "Battery Monitor" V 4600 3150 50  0000 C CNN
+F 2 "Terminal_Blocks:TerminalBlock_Pheonix_MPT-2.54mm_2pol" H 4500 3150 60  0001 C CNN
+F 3 "" H 4500 3150 60  0000 C CNN
+	1    4500 3150
+	1    0    0    1
+$EndComp
+Wire Wire Line
+	4150 2100 4300 2100
+Wire Wire Line
+	4300 2100 4300 2550
+Wire Wire Line
+	4150 2000 4950 2000
+Wire Wire Line
+	5250 2000 5500 2000
+Wire Wire Line
+	5800 2000 6000 2000
+Wire Wire Line
+	6300 2000 7200 2000
+Wire Wire Line
+	5850 1550 6450 1550
+Wire Wire Line
+	6450 1550 6450 2000
+Connection ~ 6450 2000
+Wire Wire Line
+	5450 1550 4800 1550
+Wire Wire Line
+	4800 1550 4800 2000
+Connection ~ 4800 2000
+Wire Wire Line
+	7200 2100 7050 2100
+Wire Wire Line
+	7050 2100 7050 2550
+Wire Wire Line
+	4300 3100 3900 3100
+Wire Wire Line
+	4300 3200 4050 3200
+Wire Wire Line
+	4050 3200 4050 3450
+$Comp
+L GND #PWR03
+U 1 1 59BE3AEE
+P 4050 3450
+F 0 "#PWR03" H 4050 3200 50  0001 C CNN
+F 1 "GND" H 4050 3300 50  0000 C CNN
+F 2 "" H 4050 3450 60  0000 C CNN
+F 3 "" H 4050 3450 60  0000 C CNN
+	1    4050 3450
+	1    0    0    -1
+$EndComp
+Text Label 3900 3100 0    60   ~ 0
+VOut
+$Comp
+L CONN_01X02 P6
+U 1 1 59BE3C1B
+P 4500 4150
+F 0 "P6" H 4500 4300 50  0000 C CNN
+F 1 "Cell Monitor" V 4600 4150 50  0000 C CNN
+F 2 "Terminal_Blocks:TerminalBlock_Pheonix_MPT-2.54mm_2pol" H 4500 4150 60  0001 C CNN
+F 3 "" H 4500 4150 60  0000 C CNN
+	1    4500 4150
+	1    0    0    1
+$EndComp
+Wire Wire Line
+	4300 4100 3900 4100
+Wire Wire Line
+	4300 4200 4050 4200
+Wire Wire Line
+	4050 4200 4050 4450
+$Comp
+L GND #PWR04
+U 1 1 59BE3C24
+P 4050 4450
+F 0 "#PWR04" H 4050 4200 50  0001 C CNN
+F 1 "GND" H 4050 4300 50  0000 C CNN
+F 2 "" H 4050 4450 60  0000 C CNN
+F 3 "" H 4050 4450 60  0000 C CNN
+	1    4050 4450
+	1    0    0    -1
+$EndComp
+Text Label 3900 4100 0    60   ~ 0
+VIn
+$Comp
+L CONN_01X02 P4
+U 1 1 59BE3CE4
+P 7050 3600
+F 0 "P4" H 7050 3750 50  0000 C CNN
+F 1 "Load" V 7150 3600 50  0000 C CNN
+F 2 "tl2c-footprint:PCB_Screw_Terminal_Block_5.08mm_x_2" H 7050 3600 60  0001 C CNN
+F 3 "" H 7050 3600 60  0000 C CNN
+	1    7050 3600
+	1    0    0    1
+$EndComp
+Wire Wire Line
+	6850 3550 6450 3550
+Wire Wire Line
+	6850 3650 6600 3650
+Wire Wire Line
+	6600 3650 6600 3900
+$Comp
+L GND #PWR05
+U 1 1 59BE3CED
+P 6600 3900
+F 0 "#PWR05" H 6600 3650 50  0001 C CNN
+F 1 "GND" H 6600 3750 50  0000 C CNN
+F 2 "" H 6600 3900 60  0000 C CNN
+F 3 "" H 6600 3900 60  0000 C CNN
+	1    6600 3900
+	1    0    0    -1
+$EndComp
+Text Label 5850 3550 0    60   ~ 0
+VOut
+$Comp
+L CONN_01X02 P3
+U 1 1 59BE3D5C
+P 6400 3350
+F 0 "P3" H 6400 3500 50  0000 C CNN
+F 1 "Load Power" V 6500 3350 50  0000 C CNN
+F 2 "tl2c-footprint:PCB_Screw_Terminal_Block_5.08mm_x_2" H 6400 3350 60  0001 C CNN
+F 3 "" H 6400 3350 60  0000 C CNN
+	1    6400 3350
+	0    1    -1   0
+$EndComp
+Wire Wire Line
+	6350 3550 5850 3550
 $EndSCHEMATC
